Commit message: 调试环境基本搭好，准备对齐数据

File: depoly/src/unitree_ros-master/robots/go2_description/xacro/robot.xacro (robot description, xacro)
@@ -56,4 +56,58 @@
         </inertial>
     </link>
+    <!-- 支架 -->
+    <link name="pillar">
+        <visual>
+        <origin rpy="0 0 0" xyz="0 0 -0.3"/>
+        <geometry>
+            <box size="0.1 0.1 0.5"/>
+        </geometry>
+        <material name="orange"/>
+        </visual>
+        <collision>
+        <origin rpy="0 0 0" xyz="0 0 -0.3"/>
+        <geometry>
+            <box size="0.1 0.1 0.5"/>
+        </geometry>
+        </collision>
+        <inertial>
+        <origin rpy="0 0 0" xyz="0.012731 0.002186 0.000515"/>
+        <mass value="5"/>
+        <inertia ixx="0.01683993" ixy="8.3902e-05" ixz="0.000597679" iyy="0.056579028" iyz="2.5134e-05" izz="0.064713601"/>
+        </inertial>
+    </link>
+    <!-- Joint connecting trunk to pillar -->
+    <joint name="trunk_to_pillar_joint" type="fixed">
+        <parent link="trunk"/>
+        <child link="pillar"/>
+        <origin rpy="0 0 0" xyz="0 0 0"/>
+    </joint>
+    <!-- bottom link-->
+    <link name="bottom">
+        <visual>
+        <origin rpy="0 0 0" xyz="0 0 -0.6"/>
+        <geometry>
+            <box size="1 1 0.1"/>
+        </geometry>
+        <material name="orange"/>
+        </visual>
+        <collision>
+        <origin rpy="0 0 0" xyz="0 0 -0.6"/>
+        <geometry>
+            <box size="1 1 0.1"/>
+        </geometry>
+        </collision>
+        <inertial>
+        <origin rpy="0 0 0" xyz="0.012731 0.002186 0.000515"/>
+        <mass value="10"/>
+        <inertia ixx="0.01683993" ixy="8.3902e-05" ixz="0.000597679" iyy="0.056579028" iyz="2.5134e-05" izz="0.064713601"/>
+        </inertial>
+    </link>
+    <joint name="trunk_to_bottom_joint" type="fixed">
+        <parent link="trunk"/>
+        <child link="bottom"/>
+        <origin rpy="0.3 0.3 0" xyz="0 0 0"/>
+    </joint>
+    <!--  支架 -->
     <joint name="imu_joint" type="fixed">
         <parent link="trunk"/>

Commit message: 勉强能run了效果不好

File: depoly/src/unitree_ros-master/robots/go2_description/xacro/robot.xacro (robot description, xacro)
@@ -56,58 +56,4 @@
         </inertial>
     </link>
-    <!-- 支架 -->
-    <link name="pillar">
-        <visual>
-        <origin rpy="0 0 0" xyz="0 0 -0.3"/>
-        <geometry>
-            <box size="0.1 0.1 0.5"/>
-        </geometry>
-        <material name="orange"/>
-        </visual>
-        <collision>
-        <origin rpy="0 0 0" xyz="0 0 -0.3"/>
-        <geometry>
-            <box size="0.1 0.1 0.5"/>
-        </geometry>
-        </collision>
-        <inertial>
-        <origin rpy="0 0 0" xyz="0.012731 0.002186 0.000515"/>
-        <mass value="5"/>
-        <inertia ixx="0.01683993" ixy="8.3902e-05" ixz="0.000597679" iyy="0.056579028" iyz="2.5134e-05" izz="0.064713601"/>
-        </inertial>
-    </link>
-    <!-- Joint connecting trunk to pillar -->
-    <joint name="trunk_to_pillar_joint" type="fixed">
-        <parent link="trunk"/>
-        <child link="pillar"/>
-        <origin rpy="0 0 0" xyz="0 0 0"/>
-    </joint>
-    <!-- bottom link-->
-    <link name="bottom">
-        <visual>
-        <origin rpy="0 0 0" xyz="0 0 -0.6"/>
-        <geometry>
-            <box size="1 1 0.1"/>
-        </geometry>
-        <material name="orange"/>
-        </visual>
-        <collision>
-        <origin rpy="0 0 0" xyz="0 0 -0.6"/>
-        <geometry>
-            <box size="1 1 0.1"/>
-        </geometry>
-        </collision>
-        <inertial>
-        <origin rpy="0 0 0" xyz="0.012731 0.002186 0.000515"/>
-        <mass value="10"/>
-        <inertia ixx="0.01683993" ixy="8.3902e-05" ixz="0.000597679" iyy="0.056579028" iyz="2.5134e-05" izz="0.064713601"/>
-        </inertial>
-    </link>
-    <joint name="trunk_to_bottom_joint" type="fixed">
-        <parent link="trunk"/>
-        <child link="bottom"/>
-        <origin rpy="0.3 0.3 0" xyz="0 0 0"/>
-    </joint>
-    <!--  支架 -->
     <joint name="imu_joint" type="fixed">
         <parent link="trunk"/>
